File: network.sch (KiCad schematic (older format))
At the start: 0 parts

Commit message: some work on the network section
Parts:
- added C?: C, ~, symbol C
- added R? (x6): 10k, ~, symbol R
- added R?: 1k, ~, symbol R
- added R?: 4k99, ~, symbol R
- added R? (x3): 4k7, ~, symbol R
- added U?: KSZ9021RL, symbol KSZ9021RL
Connections:
- new net: R?.2, U?.43 (RX_DV/CLK125_EN)
- new net: C?.1, R?.2, U?.56 (RXD3/MODE3)
- new net: R?.1, U?.62 (ISET)
- new net DVDDH: R?.1, R?.1, R?.1, R?.1, R?.1, R?.1, R?.2, R?.2, R?.2
- new net GND: C?.2, R?.2, R?.2, U?.17 (VSS), U?.18 (VSS), U?.23 (VSS), U?.28 (VSS), U?.3 (AGNDH), U?.34 (VSS), U?.39 (VSS), U?.53 (VSS), U?.63 (AGNDH_BG), U?.65 (PAD), U?.9 (AGNDH)
- new net PHY_CLK125: R?.1, U?.55 (CLK25_NDO/LED_MODE)
- new net PHY_INT_N: R?.1, U?.51 (INT_N)
- new net PHY_MDC: U?.48 (MDC)
- new net PHY_MDIO: R?.1, U?.49 (MDIO)
- new net PHY_RXD0: R?.2, U?.42 (RXD0/MODE0)
- new net PHY_RXD1: R?.2, U?.41 (RXD1/MODE1)
- new net PHY_RXD2: R?.2, U?.58 (RXD2/MODE2)
- new net PHY_RXD3: R?.2, U?.56 (RXD3/MODE3)
- new net PHY_RX_CLK: R?.1, U?.46 (RX_CLK/PHYAD2)
- new net PHY_TXD0: U?.24 (TXD0)
- new net PHY_TXD1: U?.25 (TXD1)
- new net PHY_TXD2: U?.26 (TXD2)
- new net PHY_TXD3: U?.27 (TXD3)
- new net PHY_TX_CLK: U?.32 (GTX_CLK)
- new net PHY_TX_EN: U?.33 (TX_EN)

Commit message: more work on networking
Parts:
- added C? (x5): 100nF, ~, symbol C
- added R?: 1k, ~, symbol R
- added R?: 10k, ~, symbol R
- added R? (x2): 120, ~, symbol R
- added U?: 0821-1X1T-43-F, symbol 0821-1X1T-43-F
Connections:
- net DVDDH is gone; now on net +3.3V: R?.1, R?.1, R?.1, R?.1, R?.1, R?.1, R?.2, R?.2, R?.2
- net GND: now also C?.1, C?.1, C?.1, C?.1, C?.2, R?.2, U?.20 (GND), U?.21 (SHIELD)
- net at U?.1 (TXRXP_A): now also U?.11 (TRD1+)
- net at U?.10 (TXRXP_C): now also U?.3 (TRD3+)
- net at U?.11 (TXRXM_C): now also U?.2 (TRD3-)
- net at U?.14 (TXRXP_D): now also U?.8 (TRD4+)
- net at U?.15 (TXRXM_D): now also U?.9 (TRD4-)
- net at U?.19 (LED2/PHYAD1): now also R?.1, U?.13 (LED1)
- net at U?.2 (TXRXM_A): now also U?.10 (RTD1-)
- net +3.3V: now reaches U?.20 (DVDDH)
- net +3.3V: now also U?.30 (DVDDH), U?.37 (DVDDH), U?.44 (DVDDH), C?.1, R?.2, R?.2, R?.2
- net at U?.21 (LED1/PHYAD0): now also R?.1, U?.15 (LED2)
- net at U?.7 (TXRXP_B): now also U?.4 (TRD2+)
- net at U?.8 (TXRXM_B): now also U?.5 (TRD2-)
- new net: C?.2, U?.1 (TRCT3)
- new net: C?.2, U?.12 (TRCT1)
- new net: R?.1, U?.14
- new net: R?.1, U?.16
- new net: C?.2, U?.6 (TRCT2)
- new net: C?.2, U?.7 (TRCT4)
- new net USB_5V: U?.17 (+5V)
- new net USB_D+: U?.19 (D+)
- new net USB_D-: U?.18 (D-)
Other:
- note added: "Gigabit Ethernet"
- moved on the sheet: C?, R?, U?

Commit message: fixes
Parts:
- added U?: 25MHZXO, symbol 25MHZXO
- added U?: BAT54A, symbol BAT54A
Connections:
- net +3.3V: now also U?.1, U?.4 (VCC)
- net GND: now also U?.2 (GND)
- net at C?.1, R?.2, U?.56 (RXD3/MODE3): now also U?.3
- net CLK_25MHZ: now reaches U?.60 (XI)
- net CLK_25MHZ: now also U?.3 (OUT)
- new net PHY_RESET_N: U?.2
