File: power.sch (KiCad schematic (older format))
At the start: 0 parts

Commit message: tx/rx section mostly complete
Parts:
- added C? (x7): C, symbol C
- added R? (x2): R, symbol R
- added R?: JMP1, symbol R
- added U?: MAX6126A21, symbol MAX6126A21
Connections:
- new net: C?.1, U?.1 (NR)
- new net: C?.1, R?.1, R?.1, U?.6 (OUTS), U?.7 (OUTF)
- new net: C?.1, C?.1, R?.2 (x2)
- new net +5V: C?.1, U?.2 (IN)
- new net GND: C?.2, C?.2, C?.2, C?.2, C?.2, C?.2, C?.2, R?.1, R?.2, U?.3 (GND), U?.4 (GNDS)
Other:
- note added: "Ultra Low Noise Supply"

Commit message: finished rx section started on power
Parts:
- added C? (x4): C, ~, symbol C
- added R? (x6): R, ~, symbol R
- added U? (x2): MAX4477AUA, symbol MAX4477AUA
Connections:
- net GND: now also C?.2, C?.2; no longer C?.2, R?.1, U?.4 (GNDS)
- net at C?.1, C?.1, R?.2: now also U?.6
- net at C?.1, C?.1, R?.2: now also U?.2
- new net: R?.1, R?.2, U?.3
- new net: R?.1, R?.2, U?.5
- new net: C?.1, R?.1, R?.2 (x2)
- new net: C?.1, R?.1 (x2)
- new net AGND: C?.2, C?.2, C?.2, R?.1, R?.2, R?.2, U?.4 (GNDS)
Other:
- moved on the sheet: C?, R?, U?
