File: transmitter.sch (KiCad schematic (older format))
At the start: 0 parts

Commit message: tx/rx section mostly complete
Parts:
- added C? (x9): 100n, symbol C
- added C? (x3): C, symbol C
- added C? (x2): 56p, symbol C
- added C?: 3p3, symbol C
- added C?: 22p, symbol C
- added C?: 2p2, symbol C
- added C?: 8p2, symbol C
- added C?: 6p8, symbol C
- added C?: 18p, symbol C
- added C?: 1n, symbol C
- added L? (x2): 120nH, symbol INDUCTOR
- added L?: 150nH, symbol INDUCTOR
- added L?: 15uH, symbol INDUCTOR
- added L?: INDUCTOR, symbol INDUCTOR
- added R?: JMP3, symbol R
- added R?: 180, symbol R
- added R?: 2k, symbol R
- added R?: 1k8, symbol R
- added R?: 1k5, symbol R
- added R?: 1k, symbol R
- added R?: 10, symbol R
- added R? (x2): 10k, symbol R
- added U?: AD9774, symbol AD9774
- added U?: AD7801, symbol AD7801
- added U?: ADT4-6T, ~, symbol ADT4-6T
- added U?: BGA616, symbol BGA616
- added U?: TX_OUT, symbol SMA
- added U?: CVHD-950, symbol CVHD-950
Connections:
- new net: C?.2, C?.2, C?.2, R?.1, R?.1, R?.2, U?.16 (REFLO), U?.17 (AGND), U?.20 (ACOM), U?.5
- new net: C?.1, C?.1, R?.2, U?.17 (REFIO)
- new net: R?.2, U?.18 (FS_ADJ)
- new net: R?.2, U?.21 (IOUTB), U?.6
- new net: R?.1, U?.22 (IOUTA), U?.4
- new net: R?.2, U?.19 (VOUT)
- new net: C?.1, U?.3 (x2)
- new net: C?.1, R?.1, R?.1, R?.1
- new net: C?.1, C?.1, C?.2, L?.2
- new net: C?.1, C?.1, C?.1, C?.2, L?.1, L?.2
- new net: C?.1, C?.1, C?.2, L?.1, L?.2
- new net: C?.1, C?.1, C?.2, L?.1
- new net: C?.2, U?.1 (x2)
- new net: L?.2, R?.2
- new net: C?.1, C?.1, C?.1, L?.1, R?.1
- new net: C?.1, R?.1, R?.2, U?.1 (VCON)
- new net +3.3V: U?.12 (PD), U?.14 (CLR), U?.15 (VDD), U?.25 (MODE), U?.27 (DVDD)
- new net +3.3VADC: C?.1, C?.1, C?.1, R?.1, U?.16 (REFIN), U?.24 (AVDD), U?.4 (VDD)
- new net +5V: L?.2
- new net CLK122: U?.28 (CLOCK), U?.3 (OUT)
- new net GND: C?.2, C?.2, C?.2, C?.2, C?.2, C?.2, C?.2, C?.2, C?.2, C?.2, C?.2, C?.2, R?.2, R?.2, U?.1, U?.11 (DGND), U?.13 (LDAC), U?.15 (SLEEP), U?.2, U?.2, U?.2 (GND), U?.20 (DGND), U?.26 (DCOM), U?.3, U?.4
- new net LVL_CS: U?.9 (CS)
- new net LVL_DB0: U?.8 (DB0)
- new net LVL_DB1: U?.7 (DB1)
- new net LVL_DB2: U?.6 (DB2)
- new net LVL_DB3: U?.5 (DB3)
- new net LVL_DB4: U?.4 (DB4)
- new net LVL_DB5: U?.3 (DB5)
- new net LVL_DB6: U?.2 (DB6)
- new net LVL_DB7: U?.1 (DB7)
- new net LVL_WR: U?.10 (WR)
- new net TX_DB0: U?.14 (DB0)
- new net TX_DB1: U?.13 (DB1)
- new net TX_DB10: U?.4 (DB10)
- new net TX_DB11: U?.3 (DB11)
- new net TX_DB12: U?.2 (DB12)
- new net TX_DB13: U?.1 (DB13)
- new net TX_DB2: U?.12 (DB2)
- new net TX_DB3: U?.11 (DB3)
- new net TX_DB4: U?.10 (DB4)
- new net TX_DB5: U?.9 (DB5)
- new net TX_DB6: U?.8 (DB6)
- new net TX_DB7: U?.7 (DB7)
- new net TX_DB8: U?.6 (DB8)
- new net TX_DB9: U?.5 (DB9)
Other:
- note added: "Level Control"
- note added: "Low Pass Filter (70Mhz)"
- note added: "MMIC"
- note added: "Master Oscillator"
- note added: "TX DAC"

Commit message: finished rx section started on power
Parts:
- L?: value INDUCTOR -> BLM21AG331SN1

Commit message: additions and fixes
Parts:
- L?: value 15uH -> 2.2uH
- R?: value 2k -> 3k9
